File: hardware/cs107e-ps2board/basic board.sch (EAGLE design)
At the start: 7 parts

Commit message: added screencasts to schedule commit 5d7a2d36071142bcfbe455836e15ba197b9dce1a Author: Chris Gregg <tofergregg@gmail.com> Date:   Wed Oct 3 08:20:51 2018 -0700
    added screencasts to schedule
Parts:
- added R2: 1000, resistor:R-US_0309/12
Connections:
- net N$3: now also R2.2
- net N$5: now also R2.1
Changed lines of the file:
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@@
 <?xml version="1.0" encoding="utf-8"?>
 <!DOCTYPE eagle SYSTEM "eagle.dtd">
-<eagle version="8.7.0">
+<eagle version="9.1.3">
 <drawing>
 <settings>
@@
 <part name="RESET" library="switch" library_urn="urn:adsk.eagle:library:380" deviceset="55?-1LED" device="01" package3d_urn="urn:adsk.eagle:package:27757/1"/>
 <part name="R1" library="resistor" library_urn="urn:adsk.eagle:library:348" deviceset="R-US_" device="0309/12" package3d_urn="urn:adsk.eagle:package:26089/1" value="1000"/>
+<part name="R2" library="resistor" library_urn="urn:adsk.eagle:library:348" deviceset="R-US_" device="0309/12" package3d_urn="urn:adsk.eagle:package:26089/1" value="1000"/>
 </parts>
 <sheets>
@@
 <instance part="RESET" gate="-LED" x="53.34" y="12.7" rot="R90"/>
 <instance part="R1" gate="G$1" x="30.48" y="12.7"/>
+<instance part="R2" gate="G$1" x="73.66" y="33.02"/>
 </instances>
 <busses>
@@
 <pinref part="DATA" gate="G$1" pin="1"/>
 <wire x1="71.12" y1="35.56" x2="78.74" y2="35.56" width="0.1524" layer="91"/>
+<pinref part="R2" gate="G$1" pin="2"/>
+<wire x1="78.74" y1="35.56" x2="78.74" y2="33.02" width="0.1524" layer="91"/>
+<junction x="78.74" y="35.56"/>
 </segment>
 </net>
@@
 <pinref part="RESET" gate="-1" pin="NO"/>
 <pinref part="5V" gate="G$1" pin="1"/>
-<wire x1="43.18" y1="25.4" x2="78.74" y2="25.4" width="0.1524" layer="91"/>
-</segment>
-</net>
+<wire x1="43.18" y1="25.4" x2="68.58" y2="25.4" width="0.1524" layer="91"/>
+<pinref part="R2" gate="G$1" pin="1"/>
+<wire x1="68.58" y1="25.4" x2="78.74" y2="25.4" width="0.1524" layer="91"/>
+<wire x1="68.58" y1="33.02" x2="68.58" y2="25.4" width="0.1524" layer="91"/>
+<junction x="68.58" y="25.4"/>
+</segment>
+</net>
