File: hardware/cs107e-ps2board/basic board.brd (EAGLE design)
At the start: 20.2 x 41.9 mm, 7 parts

Commit message: added screencasts to schedule commit 5d7a2d36071142bcfbe455836e15ba197b9dce1a Author: Chris Gregg <tofergregg@gmail.com> Date:   Wed Oct 3 08:20:51 2018 -0700
    added screencasts to schedule
Parts:
- added R2: 1000, resistor:0309/12
- moved R1 3.56 mm to (18.0, 62.1)
Connections:
- net N$3: now also R2.2
- net N$5: now also R2.1
Routing:
- net N$3: track 27.2 -> 49.7 mm
- net N$5: track 18.7 -> 35.0 mm
- net N$6: track 11.5 -> 15.0 mm
- net N$7: track 6.13 -> 7.98 mm
Changed lines of the file:
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@@
 <?xml version="1.0" encoding="utf-8"?>
 <!DOCTYPE eagle SYSTEM "eagle.dtd">
-<eagle version="8.7.0">
+<eagle version="9.1.3">
 <drawing>
 <settings>
@@
 <param name="checkStop" value="0"/>
 <param name="checkValues" value="0"/>
+<param name="checkNames" value="1"/>
+<param name="checkWireStubs" value="1"/>
+<param name="checkPolygonWidth" value="0"/>
 <param name="useDiameter" value="13"/>
 <param name="maxErrors" value="50"/>
@@
 <attribute name="VALUE" x="3.81" y="76.98" size="1.778" layer="27" ratio="10"/>
 </element>
-<element name="R1" library="resistor" library_urn="urn:adsk.eagle:library:348" package="0309/12" package3d_urn="urn:adsk.eagle:package:26089/1" value="1000" x="18" y="58.54" smashed="yes" rot="R270">
-<attribute name="NAME" x="15.905" y="51.731" size="1.27" layer="21" ratio="10" rot="R270"/>
-<attribute name="VALUE" x="17.3142" y="60.715" size="1.27" layer="21" ratio="10" rot="R270"/>
-</element>
+<element name="R1" library="resistor" library_urn="urn:adsk.eagle:library:348" package="0309/12" package3d_urn="urn:adsk.eagle:package:26089/1" value="1000" x="18" y="62.096" smashed="yes" rot="R270">
+<attribute name="NAME" x="15.905" y="55.287" size="1.27" layer="21" ratio="10" rot="R270"/>
+<attribute name="VALUE" x="17.3142" y="64.271" size="1.27" layer="21" ratio="10" rot="R270"/>
+</element>
+<element name="R2" library="resistor" library_urn="urn:adsk.eagle:library:348" package="0309/12" package3d_urn="urn:adsk.eagle:package:26089/1" value="1000" x="17.78" y="46.228" rot="R90"/>
 </elements>
 <signals>
@@
 <wire x1="9.652" y1="44.878" x2="10.43" y2="44.1" width="0.4064" layer="1"/>
 <wire x1="9.652" y1="69.848" x2="9.652" y2="44.878" width="0.4064" layer="1"/>
+<contactref element="R2" pad="2"/>
+<wire x1="10.43" y1="44.1" x2="10.668" y2="43.862" width="0.1524" layer="16"/>
+<wire x1="10.668" y1="43.862" x2="10.668" y2="40.64" width="0.1524" layer="16"/>
+<wire x1="10.668" y1="40.64" x2="15.748" y2="40.64" width="0.1524" layer="16"/>
+<wire x1="15.748" y1="40.64" x2="15.748" y2="52.324" width="0.1524" layer="16"/>
+<wire x1="15.748" y1="52.324" x2="16.002" y2="52.578" width="0.1524" layer="16"/>
+<wire x1="16.002" y1="52.578" x2="17.78" y2="52.578" width="0.1524" layer="16"/>
 </signal>
 <signal name="N$4">
@@
 <contactref element="RESET" pad="1B"/>
 <contactref element="R1" pad="1"/>
-<wire x1="18" y1="64.89" x2="12.81" y2="57.16" width="0.4064" layer="1"/>
-<wire x1="12.81" y1="57.16" x2="12.81" y2="55" width="0.4064" layer="1"/>
+<wire x1="18" y1="68.446" x2="12.81" y2="60.716" width="0.4064" layer="1"/>
+<wire x1="12.81" y1="60.716" x2="12.81" y2="55" width="0.4064" layer="1"/>
 </signal>
 <signal name="N$7">
 <contactref element="R1" pad="2"/>
 <contactref element="RESET" pad="+"/>
-<wire x1="12.81" y1="49.92" x2="15.73" y2="49.92" width="0.4064" layer="1"/>
-<wire x1="15.73" y1="49.92" x2="18" y2="52.19" width="0.4064" layer="1"/>
+<wire x1="12.81" y1="50.556" x2="18" y2="55.746" width="0.4064" layer="1"/>
+<wire x1="12.81" y1="49.92" x2="12.81" y2="50.556" width="0.4064" layer="1"/>
 </signal>
 <signal name="PE3">
@@
 <wire x1="2.032" y1="56.896" x2="5.19" y2="60.054" width="0.4064" layer="1"/>
 <wire x1="5.19" y1="60.054" x2="5.19" y2="60.08" width="0.4064" layer="1"/>
+<contactref element="R2" pad="1"/>
+<wire x1="5.35" y1="44.1" x2="5.35" y2="40.37" width="0.1524" layer="16"/>
+<wire x1="5.842" y1="39.878" x2="17.78" y2="39.878" width="0.1524" layer="16"/>
+<wire x1="5.35" y1="40.37" x2="5.842" y2="39.878" width="0.1524" layer="16"/>
 </signal>
 </signals>
+<mfgpreviewcolors>
+<mfgpreviewcolor name="soldermaskcolor" color="0xC8008000"/>
+<mfgpreviewcolor name="silkscreencolor" color="0xFFFEFEFE"/>
+<mfgpreviewcolor name="backgroundcolor" color="0xFF282828"/>
+<mfgpreviewcolor name="coppercolor" color="0xFFFFBF00"/>
+<mfgpreviewcolor name="substratecolor" color="0xFF786E46"/>
+</mfgpreviewcolors>
 </board>
 </drawing>

Commit message: Merge branch 'master' of github.com:cs107e/staff commit c34fac17d5b98fb7d3ca4e05ab2c3df01d6cdd47 Merge: 94aee8d c70b920 Author: Chris Gregg <tofergregg@gmail.com> Date:   Sat Oct 6 12:46:18 2018 -0700
    Merge branch 'master' of github.com:cs107e/staff
Parts:
- moved R1 1.02 mm to (18.0, 63.1)
Routing:
- net N$3: track 49.7 -> 46.6 mm
- net N$6: track 15.0 -> 16.4 mm
- net N$7: track 7.98 -> 8.99 mm
Other:
- board text added: "Stanford CS107E PS/2 breakout board http://cs107e.stanford.edu Philip Levis & Chris Gregg v1.1 10/2018"
- board text removed: "Stanford CS107E PS/2 breakout board http://cs107e.stanford.edu Philip Levis & Chris Gregg v1.0 4/2018"
Changed lines of the file:
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@@
 <grid distance="20" unitdist="mil" unit="mil" style="lines" multiple="5" display="yes" altdistance="1" altunitdist="mil" altunit="mil"/>
 <layers>
-<layer number="1" name="Top" color="4" fill="1" visible="no" active="yes"/>
+<layer number="1" name="Top" color="4" fill="1" visible="yes" active="yes"/>
 <layer number="16" name="Bottom" color="1" fill="1" visible="yes" active="yes"/>
 <layer number="17" name="Pads" color="2" fill="1" visible="yes" active="yes"/>
@@
 http://cs107e.stanford.edu
 Philip Levis &amp; Chris Gregg
-v1.0 4/2018</text>
+v1.1 10/2018</text>
 </plain>
 <attributes>
@@
 <attribute name="VALUE" x="3.81" y="76.98" size="1.778" layer="27" ratio="10"/>
 </element>
-<element name="R1" library="resistor" library_urn="urn:adsk.eagle:library:348" package="0309/12" package3d_urn="urn:adsk.eagle:package:26089/1" value="1000" x="18" y="62.096" smashed="yes" rot="R270">
-<attribute name="NAME" x="15.905" y="55.287" size="1.27" layer="21" ratio="10" rot="R270"/>
-<attribute name="VALUE" x="17.3142" y="64.271" size="1.27" layer="21" ratio="10" rot="R270"/>
-</element>
-<element name="R2" library="resistor" library_urn="urn:adsk.eagle:library:348" package="0309/12" package3d_urn="urn:adsk.eagle:package:26089/1" value="1000" x="17.78" y="46.228" rot="R90"/>
+<element name="R1" library="resistor" library_urn="urn:adsk.eagle:library:348" package="0309/12" package3d_urn="urn:adsk.eagle:package:26089/1" value="1000" x="18" y="63.112" smashed="yes" rot="R270">
+<attribute name="NAME" x="15.905" y="56.303" size="1.27" layer="21" ratio="10" rot="R270"/>
+<attribute name="VALUE" x="17.3142" y="65.287" size="1.27" layer="21" ratio="10" rot="R270"/>
+</element>
+<element name="R2" library="resistor" library_urn="urn:adsk.eagle:library:348" package="0309/12" package3d_urn="urn:adsk.eagle:package:26089/1" value="1000" x="17.78" y="46.228" smashed="yes" rot="R90">
+<attribute name="NAME" x="15.875" y="42.037" size="1.27" layer="25" ratio="10" rot="R90"/>
+<attribute name="VALUE" x="18.4658" y="44.069" size="1.27" layer="21" ratio="10" rot="R90"/>
+</element>
 </elements>
 <signals>
@@
 <wire x1="9.652" y1="69.848" x2="9.652" y2="44.878" width="0.4064" layer="1"/>
 <contactref element="R2" pad="2"/>
-<wire x1="10.43" y1="44.1" x2="10.668" y2="43.862" width="0.1524" layer="16"/>
-<wire x1="10.668" y1="43.862" x2="10.668" y2="40.64" width="0.1524" layer="16"/>
-<wire x1="10.668" y1="40.64" x2="15.748" y2="40.64" width="0.1524" layer="16"/>
-<wire x1="15.748" y1="40.64" x2="15.748" y2="52.324" width="0.1524" layer="16"/>
-<wire x1="15.748" y1="52.324" x2="16.002" y2="52.578" width="0.1524" layer="16"/>
-<wire x1="16.002" y1="52.578" x2="17.78" y2="52.578" width="0.1524" layer="16"/>
+<wire x1="17.78" y1="52.578" x2="15.748" y2="50.546" width="0.4064" layer="16"/>
+<wire x1="15.748" y1="50.546" x2="15.748" y2="41.656" width="0.4064" layer="16"/>
+<wire x1="15.748" y1="41.656" x2="10.668" y2="41.656" width="0.4064" layer="16"/>
+<wire x1="10.43" y1="41.894" x2="10.668" y2="41.656" width="0.4064" layer="16"/>
+<wire x1="10.43" y1="44.1" x2="10.43" y2="41.894" width="0.4064" layer="16"/>
 </signal>
 <signal name="N$4">
@@
 <contactref element="RESET" pad="1B"/>
 <contactref element="R1" pad="1"/>
-<wire x1="18" y1="68.446" x2="12.81" y2="60.716" width="0.4064" layer="1"/>
-<wire x1="12.81" y1="60.716" x2="12.81" y2="55" width="0.4064" layer="1"/>
+<wire x1="18" y1="69.462" x2="15.858" y2="66.2717" width="0.4064" layer="1"/>
+<wire x1="15.858" y1="66.2717" x2="15.858" y2="58.048" width="0.4064" layer="1"/>
+<wire x1="15.858" y1="58.048" x2="12.81" y2="55" width="0.4064" layer="1"/>
 </signal>
 <signal name="N$7">
 <contactref element="R1" pad="2"/>
 <contactref element="RESET" pad="+"/>
-<wire x1="12.81" y1="50.556" x2="18" y2="55.746" width="0.4064" layer="1"/>
-<wire x1="12.81" y1="49.92" x2="12.81" y2="50.556" width="0.4064" layer="1"/>
+<wire x1="12.81" y1="51.572" x2="18" y2="56.762" width="0.4064" layer="1"/>
+<wire x1="12.81" y1="49.92" x2="12.81" y2="51.572" width="0.4064" layer="1"/>
 </signal>
 <signal name="PE3">
@@
 <wire x1="5.19" y1="60.054" x2="5.19" y2="60.08" width="0.4064" layer="1"/>
 <contactref element="R2" pad="1"/>
-<wire x1="5.35" y1="44.1" x2="5.35" y2="40.37" width="0.1524" layer="16"/>
-<wire x1="5.842" y1="39.878" x2="17.78" y2="39.878" width="0.1524" layer="16"/>
-<wire x1="5.35" y1="40.37" x2="5.842" y2="39.878" width="0.1524" layer="16"/>
+<wire x1="17.78" y1="39.878" x2="17.526" y2="39.624" width="0.4064" layer="16"/>
+<wire x1="17.526" y1="39.624" x2="6.096" y2="39.624" width="0.4064" layer="16"/>
+<wire x1="6.096" y1="39.624" x2="5.35" y2="40.37" width="0.4064" layer="16"/>
+<wire x1="5.35" y1="40.37" x2="5.35" y2="44.1" width="0.4064" layer="16"/>
 </signal>
 </signals>
